File: MySXSenors.brd (EAGLE design)
At the start: 25.4 x 35.6 mm, 6 parts

Commit message: add uart
Parts:
- added UART: (no value), con-lstb:MA04-1
Connections:
- net D1_DFM: now also UART.2
- net D2_DTM: now also UART.1
- net D3_INT: no longer PIR2.2
- net D4_INT: now also PIR2.2
- net GND: now also ISP.6, UART.3; no longer ISP.2
- net VCC: now also ISP.2, UART.4; no longer ISP.6
Routing:
- net D1_DFM: track 0.00 -> 26.0 mm, vias 0 -> 1
- net D3_INT: track 22.2 -> 0.00 mm
- net D2_DTM: track 0.00 -> 21.3 mm
- net D4_INT: track 0.00 -> 20.0 mm
- net GND: track 49.9 -> 59.7 mm
- net D8_SDA: track 19.8 -> 21.0 mm
- net D7_SCL: track 26.3 -> 27.2 mm
Other:
- outline, holes or cut-outs redrawn
- board text added: "MySX Multisensor 1.1"

Commit message: make MysX connector smd mounted
Parts:
- removed PIR1: (no value), pinhead:1X01
- removed X1: (no value), con-lsta:FE10-2
- added SV1: (no value), my-con-lsta:FE10-2
Connections:
- net D10_A4: now also SV1.15; no longer X1.16
- net D11_MOSI: now also SV1.18; no longer X1.17
- net D12_MISO: now also SV1.17; no longer X1.18
- net D13_SCK: now also SV1.20; no longer X1.19
- net D14_CS: now also SV1.19; no longer X1.20
- net D1_DFM: now also SV1.6; no longer X1.5
- net D2_DTM: now also SV1.5; no longer X1.6
- net D3_INT: now also SV1.10; no longer X1.9
- net D4_INT: now also SV1.9; no longer X1.10
- net D5_PWM: now also SV1.12; no longer X1.11
- net D6_PWM: now also SV1.11; no longer X1.12
- net D7_SCL: now also SV1.14; no longer X1.13
- net D8_SDA: now also SV1.13; no longer X1.14
- net D9_A3: now also SV1.16; no longer X1.15
- net GND: now also SV1.3; no longer X1.4
- net LEGACY_ID: now also SV1.7; no longer X1.8
- net RST: now also SV1.8; no longer X1.7
- net VCC: now also SV1.1; no longer PIR1.1, X1.2
- net VCCIO: now also SV1.4; no longer X1.3
- net VRAW: now also PIR2.1, SV1.2; no longer X1.1
Routing:
- net VRAW: track 0.00 -> 33.3 mm, vias 0 -> 3
- net VCC: track 62.7 -> 36.7 mm
- net RST: track 16.9 -> 7.82 mm
- net GND: track 59.7 -> 60.8 mm
- net D7_SCL: track 27.2 -> 26.4 mm, vias 0 -> 1
- net D11_MOSI: track 27.5 -> 28.3 mm, vias 0 -> 1
- net D8_SDA: track 21.0 -> 21.4 mm, vias 0 -> 1
Other:
- board size 25.4 x 35.6 mm -> 26.4 x 35.6 mm
- board text added: "MySX Multisensor 1.2"
- board text removed: "MySX Multisensor 1.1"

Commit message: rename DTM and DTF signals
Connections:
- net D1_DFM renamed D1_TX
- net D2_DTM renamed D2_RX
Changed lines of the file:
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@@
 <wire x1="5.715" y1="24.13" x2="4.445" y2="24.13" width="0.508" layer="1"/>
-</signal>
-<signal name="D1_DFM">
-<contactref element="UART" pad="2"/>
-<contactref element="SV1" pad="6"/>
-<wire x1="8.636" y1="19.431" x2="7.747" y2="20.32" width="0.2032" layer="16"/>
-<wire x1="19.177" y1="19.431" x2="8.636" y2="19.431" width="0.2032" layer="16"/>
-<wire x1="19.812" y1="20.066" x2="19.177" y2="19.431" width="0.2032" layer="16"/>
-<wire x1="19.812" y1="22.987" x2="19.812" y2="20.066" width="0.2032" layer="16"/>
-<wire x1="20.447" y1="23.622" x2="19.812" y2="22.987" width="0.2032" layer="16"/>
-<wire x1="20.447" y1="24.384" x2="20.447" y2="23.622" width="0.2032" layer="16"/>
-<wire x1="22.098" y1="26.035" x2="20.447" y2="24.384" width="0.2032" layer="16"/>
-<wire x1="22.225" y1="26.035" x2="22.098" y2="26.035" width="0.2032" layer="16"/>
-<wire x1="3.175" y1="20.32" x2="1.905" y2="19.05" width="0.2032" layer="1"/>
-<wire x1="3.175" y1="20.32" x2="7.747" y2="20.32" width="0.2032" layer="16"/>
-<via x="3.175" y="20.32" extent="1-16" drill="0.3302"/>
 </signal>
 <signal name="RST">
@@
 <contactref element="SV1" pad="9"/>
 <wire x1="4.445" y1="14.605" x2="4.445" y2="13.97" width="0.2032" layer="16"/>
-</signal>
-<signal name="D2_DTM">
-<wire x1="19.304" y1="19.05" x2="20.193" y2="19.939" width="0.2032" layer="16"/>
-<wire x1="20.193" y1="19.939" x2="20.193" y2="22.86" width="0.2032" layer="16"/>
-<wire x1="20.193" y1="22.86" x2="20.828" y2="23.495" width="0.2032" layer="16"/>
-<contactref element="UART" pad="1"/>
-<wire x1="22.225" y1="23.495" x2="20.828" y2="23.495" width="0.2032" layer="16"/>
-<contactref element="SV1" pad="5"/>
-<wire x1="19.304" y1="19.05" x2="4.445" y2="19.05" width="0.2032" layer="16"/>
 </signal>
 <signal name="GND" class="1">
@@
 <contactref element="SV1" pad="16"/>
 </signal>
+<signal name="D1_TX">
+<contactref element="UART" pad="2"/>
+<contactref element="SV1" pad="6"/>
+<wire x1="8.636" y1="19.431" x2="7.747" y2="20.32" width="0.2032" layer="16"/>
+<wire x1="19.177" y1="19.431" x2="8.636" y2="19.431" width="0.2032" layer="16"/>
+<wire x1="19.812" y1="20.066" x2="19.177" y2="19.431" width="0.2032" layer="16"/>
+<wire x1="19.812" y1="22.987" x2="19.812" y2="20.066" width="0.2032" layer="16"/>
+<wire x1="20.447" y1="23.622" x2="19.812" y2="22.987" width="0.2032" layer="16"/>
+<wire x1="20.447" y1="24.384" x2="20.447" y2="23.622" width="0.2032" layer="16"/>
+<wire x1="22.098" y1="26.035" x2="20.447" y2="24.384" width="0.2032" layer="16"/>
+<wire x1="3.175" y1="20.32" x2="1.905" y2="19.05" width="0.2032" layer="1"/>
+<wire x1="3.175" y1="20.32" x2="7.747" y2="20.32" width="0.2032" layer="16"/>
+<via x="3.175" y="20.32" extent="1-16" drill="0.3302"/>
+<wire x1="22.098" y1="26.035" x2="22.225" y2="26.035" width="0.2032" layer="16"/>
+</signal>
+<signal name="D2_RX">
+<contactref element="UART" pad="1"/>
+<wire x1="19.304" y1="19.05" x2="20.193" y2="19.939" width="0.2032" layer="16"/>
+<wire x1="20.193" y1="19.939" x2="20.193" y2="22.86" width="0.2032" layer="16"/>
+<wire x1="20.193" y1="22.86" x2="20.828" y2="23.495" width="0.2032" layer="16"/>
+<contactref element="SV1" pad="5"/>
+<wire x1="19.304" y1="19.05" x2="4.445" y2="19.05" width="0.2032" layer="16"/>
+<wire x1="20.828" y1="23.495" x2="22.225" y2="23.495" width="0.2032" layer="16"/>
+</signal>
 </signals>
