File: MySXSensors.kicad_pcb (KiCad board)
At the start: 2 copper layers, 10 parts, among them J1 LD2410B, J2 UART, U1 BME280, U2 BH1750FVI-TR

Commit message: fix project name
Parts:
- U2: footprint MySXSenors:XDCR_BH1750FVI-TR -> MySXSensors:XDCR_BH1750FVI-TR
- X1: footprint MySXSenors:FE10-2 -> MySXSensors:FE10-2
Changed lines of the file:
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@@
     (descr "Capacitor SMD 0402 (1005 Metric), square (rectangular) end terminal, IPC_7351 nominal with elongated pad for handsoldering. (Body size source: IPC-SM-782 page 76, https://www.pcb-3d.com/wordpress/wp-content/uploads/ipc-sm-782a_amendment_1_and_2.pdf), generated with kicad-footprint-generator")
     (tags "capacitor handsolder")
-    (property "Sheetfile" "MySXSenors.kicad_sch")
+    (property "Sheetfile" "MySXSensors.kicad_sch")
     (property "Sheetname" "")
     (property "ki_description" "Unpolarized capacitor")
@@
     (descr "Through hole straight pin header, 1x05, 1.27mm pitch, single row")
     (tags "Through hole pin header THT 1x05 1.27mm single row")
-    (property "Sheetfile" "MySXSenors.kicad_sch")
+    (property "Sheetfile" "MySXSensors.kicad_sch")
     (property "Sheetname" "")
     (property "ki_description" "Generic connector, single row, 01x05, script generated (kicad-library-utils/schlib/autogen/connector/)")
@@
     (descr "LGA-8")
     (tags "lga land grid array")
-    (property "Sheetfile" "MySXSenors.kicad_sch")
+    (property "Sheetfile" "MySXSensors.kicad_sch")
     (property "Sheetname" "")
     (property "ki_description" "3-in-1 sensor, humidity, pressure, temperature, I2C and SPI interface, 1.71-3.6V, LGA-8")
@@
     (descr "Resistor SMD 0603 (1608 Metric), square (rectangular) end terminal, IPC_7351 nominal, (Body size source: IPC-SM-782 page 72, https://www.pcb-3d.com/wordpress/wp-content/uploads/ipc-sm-782a_amendment_1_and_2.pdf), generated with kicad-footprint-generator")
     (tags "resistor")
-    (property "Sheetfile" "MySXSenors.kicad_sch")
+    (property "Sheetfile" "MySXSensors.kicad_sch")
     (property "Sheetname" "")
     (property "ki_description" "Resistor")
@@
     )
   )
-  (footprint "MySXSenors:XDCR_BH1750FVI-TR" (layer "F.Cu")
+  (footprint "MySXSensors:XDCR_BH1750FVI-TR" (layer "F.Cu")
     (at 126.15 90.525)
     (property "Availability" "")
@@
     (property "Purchase-URL" "")
     (property "STANDARD" "")
-    (property "Sheetfile" "MySXSenors.kicad_sch")
+    (property "Sheetfile" "MySXSensors.kicad_sch")
     (property "Sheetname" "")
     (property "SnapEDA_Link" "")
@@
     (descr "Capacitor SMD 0402 (1005 Metric), square (rectangular) end terminal, IPC_7351 nominal with elongated pad for handsoldering. (Body size source: IPC-SM-782 page 76, https://www.pcb-3d.com/wordpress/wp-content/uploads/ipc-sm-782a_amendment_1_and_2.pdf), generated with kicad-footprint-generator")
     (tags "capacitor handsolder")
-    (property "Sheetfile" "MySXSenors.kicad_sch")
+    (property "Sheetfile" "MySXSensors.kicad_sch")
     (property "Sheetname" "")
     (property "ki_description" "Unpolarized capacitor")
@@
     )
   )
-  (footprint "MySXSenors:FE10-2" (layer "F.Cu")
+  (footprint "MySXSensors:FE10-2" (layer "F.Cu")
     (at 137.35 112)
     (descr "<b>FEMALE HEADER</b>")
-    (property "Sheetfile" "MySXSenors.kicad_sch")
+    (property "Sheetfile" "MySXSensors.kicad_sch")
     (property "Sheetname" "")
     (property "ki_description" "Generic connector, double row, 02x10, odd/even pin numbering scheme (row 1 odd numbers, row 2 even numbers), script generated (kicad-library-utils/schlib/autogen/connector/)")
@@
     (descr "Capacitor SMD 0402 (1005 Metric), square (rectangular) end terminal, IPC_7351 nominal with elongated pad for handsoldering. (Body size source: IPC-SM-782 page 76, https://www.pcb-3d.com/wordpress/wp-content/uploads/ipc-sm-782a_amendment_1_and_2.pdf), generated with kicad-footprint-generator")
     (tags "capacitor handsolder")
-    (property "Sheetfile" "MySXSenors.kicad_sch")
+    (property "Sheetfile" "MySXSensors.kicad_sch")
     (property "Sheetname" "")
     (property "ki_description" "Unpolarized capacitor")
@@
     (descr "Through hole angled pin header, 1x04, 2.54mm pitch, 6mm pin length, single row")
     (tags "Through hole angled pin header THT 1x04 2.54mm single row")
-    (property "Sheetfile" "MySXSenors.kicad_sch")
+    (property "Sheetfile" "MySXSensors.kicad_sch")
     (property "Sheetname" "")
     (property "ki_description" "Generic connector, single row, 01x04, script generated (kicad-library-utils/schlib/autogen/connector/)")
@@
     (descr "Resistor SMD 0603 (1608 Metric), square (rectangular) end terminal, IPC_7351 nominal, (Body size source: IPC-SM-782 page 72, https://www.pcb-3d.com/wordpress/wp-content/uploads/ipc-sm-782a_amendment_1_and_2.pdf), generated with kicad-footprint-generator")
     (tags "resistor")
-    (property "Sheetfile" "MySXSenors.kicad_sch")
+    (property "Sheetfile" "MySXSensors.kicad_sch")
     (property "Sheetname" "")
     (property "ki_description" "Resistor")

Commit message: version 1.0
Parts:
- moved U2 45.4 mm to (159.7, 121.2)
- moved R2 30.0 mm to (159.2, 119.0), turned to 180 degrees
- moved R1 29.2 mm to (156.6, 118.2), turned to 90 degrees
- moved C3 28.1 mm to (159.6, 123.0), turned to 180 degrees
- moved C2 26.8 mm to (156.9, 121.2), turned to -90 degrees
- moved J1 21.2 mm to (148.4, 121.9), turned to 90 degrees
- moved C1 16.1 mm to (159.3, 96.0), turned to 180 degrees
- moved U1 13.8 mm to (159.6, 98.4)
- moved J2 12.9 mm to (146.1, 93.5), turned to 180 degrees
- moved X1 2.23 mm to (139.5, 111.4), turned to -90 degrees
Connections:
- J1 pad 1: VRAW -> D3_INT
- J1 pad 2: GND -> Net-(J1-Pin_2)
- J1 pad 4: Net-(J1-Pin_4) -> GND
- J1 pad 5: D3_INT -> VRAW
- J2 pad 1: VRAW -> Net-(J1-Pin_2)
- J2 pad 2: GND -> Net-(J1-Pin_3)
- J2 pad 3: Net-(J1-Pin_3) -> GND
- J2 pad 4: Net-(J1-Pin_4) -> VRAW
Routing:
- net GND: track 0.00 -> 80.8 mm, vias 0 -> 2
- net VCCIO: track 0.00 -> 78.8 mm, vias 0 -> 2
- net D7_SCL: track 0.00 -> 56.9 mm
- net D8_SDA: track 0.00 -> 54.6 mm, vias 0 -> 2
- net VRAW: track 0.00 -> 47.4 mm
- net Net-(J1-Pin_3): track 0.00 -> 33.0 mm
- net Net-(J1-Pin_2): track 0.00 -> 29.9 mm
- net D3_INT: track 0.00 -> 19.1 mm
- net Net-(U2-ADDR): track 0.00 -> 6.13 mm
- net Net-(U2-DVI): track 0.00 -> 4.91 mm
- added copper zone on B.Cu, net GND
- added copper zone on F.Cu, net GND
Other:
- board outline added: 27.7 x 44 mm
- board text added: "MySXSensors v1.0"
- board text added: "TX↑ RX↓GDN 5V"
