File: MySXSensors.kicad_pcb (KiCad board)
At the start: 2 copper layers, 27.7 x 44 mm, 10 parts, among them J1 LD2410B, J2 UART, U1 BME280, U2 BH1750FVI-TR

Commit message: add gas sensor
Parts:
- added U3: MQ-6, Sensor:MQ-6, F.Cu at (148.5, 95.7)
- added U4: LIS3DH, Package_LGA:LGA-16_3x3mm_P0.5mm_LayoutBorder3x5y, F.Cu at (157.0, 107.8)
Connections:
- net D12_MISO renamed D12_MISO_1
- net D13_SCK renamed D13_SCK_1
- net D2_RX renamed D2_RX_1
- net D9_A3 renamed D9_A3_1
- net VCC renamed VCC_1
