File: MySXSensors.kicad_sch (KiCad schematic)
At the start: 10 parts, among them J1 LD2410B, J2 UART, U1 BME280, U2 BH1750FVI-TR

Commit message: fix project name
Parts:
- U2: footprint MySXSenors:XDCR_BH1750FVI-TR -> MySXSensors:XDCR_BH1750FVI-TR
- X1: footprint MySXSenors:FE10-2 -> MySXSensors:FE10-2
Changed lines of the file:
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@@
     (pin "1")
     (instances
-      (project "MySXSenors"
+      (project "MySXSensors"
         (path "/95f78fe7-75c4-427a-aee1-7170190425b2"
           (reference "#PWR08") (unit 1)
@@
     (pin "4")
     (instances
-      (project "MySXSenors"
+      (project "MySXSensors"
         (path "/95f78fe7-75c4-427a-aee1-7170190425b2"
           (reference "J2") (unit 1)
@@
     (pin "1")
     (instances
-      (project "MySXSenors"
+      (project "MySXSensors"
         (path "/95f78fe7-75c4-427a-aee1-7170190425b2"
           (reference "#FLG01") (unit 1)
@@
     (pin "2")
     (instances
-      (project "MySXSenors"
+      (project "MySXSensors"
         (path "/95f78fe7-75c4-427a-aee1-7170190425b2"
           (reference "C3") (unit 1)
@@
     (pin "1")
     (instances
-      (project "MySXSenors"
+      (project "MySXSensors"
         (path "/95f78fe7-75c4-427a-aee1-7170190425b2"
           (reference "R2") (unit 1)
@@
     (pin "1")
     (instances
-      (project "MySXSenors"
+      (project "MySXSensors"
         (path "/95f78fe7-75c4-427a-aee1-7170190425b2"
           (reference "#PWR03") (unit 1)
@@
     (pin "1")
     (instances
-      (project "MySXSenors"
+      (project "MySXSensors"
         (path "/95f78fe7-75c4-427a-aee1-7170190425b2"
           (reference "R1") (unit 1)
@@
     (pin "1")
     (instances
-      (project "MySXSenors"
+      (project "MySXSensors"
         (path "/95f78fe7-75c4-427a-aee1-7170190425b2"
           (reference "#PWR05") (unit 1)
@@
     (pin "6")
     (instances
-      (project "MySXSenors"
+      (project "MySXSensors"
         (path "/95f78fe7-75c4-427a-aee1-7170190425b2"
           (reference "U1") (unit 1)
@@
     (pin "2")
     (instances
-      (project "MySXSenors"
+      (project "MySXSensors"
         (path "/95f78fe7-75c4-427a-aee1-7170190425b2"
           (reference "C1") (unit 1)
@@
     (pin "1")
     (instances
-      (project "MySXSenors"
+      (project "MySXSensors"
         (path "/95f78fe7-75c4-427a-aee1-7170190425b2"
           (reference "#PWR02") (unit 1)
@@
       (effects (font (size 1.27 1.27)))
     )
-    (property "Footprint" "MySXSenors:XDCR_BH1750FVI-TR" (at 175.895 47.625 0)
+    (property "Footprint" "MySXSensors:XDCR_BH1750FVI-TR" (at 175.895 47.625 0)
       (effects (font (size 1.27 1.27)) (justify bottom) hide)
     )
@@
     (pin "5")
     (instances
-      (project "MySXSenors"
+      (project "MySXSensors"
         (path "/95f78fe7-75c4-427a-aee1-7170190425b2"
           (reference "U2") (unit 1)
@@
     (pin "1")
     (instances
-      (project "MySXSenors"
+      (project "MySXSensors"
         (path "/95f78fe7-75c4-427a-aee1-7170190425b2"
           (reference "#PWR07") (unit 1)
@@
     (pin "1")
     (instances
-      (project "MySXSenors"
+      (project "MySXSensors"
         (path "/95f78fe7-75c4-427a-aee1-7170190425b2"
           (reference "#PWR04") (unit 1)
@@
     (pin "1")
     (instances
-      (project "MySXSenors"
+      (project "MySXSensors"
         (path "/95f78fe7-75c4-427a-aee1-7170190425b2"
           (reference "#PWR01") (unit 1)
@@
     (pin "5")
     (instances
-      (project "MySXSenors"
+      (project "MySXSensors"
         (path "/95f78fe7-75c4-427a-aee1-7170190425b2"
           (reference "J1") (unit 1)
@@
     (pin "1")
     (instances
-      (project "MySXSenors"
+      (project "MySXSensors"
         (path "/95f78fe7-75c4-427a-aee1-7170190425b2"
           (reference "#FLG02") (unit 1)
@@
     (pin "1")
     (instances
-      (project "MySXSenors"
+      (project "MySXSensors"
         (path "/95f78fe7-75c4-427a-aee1-7170190425b2"
           (reference "#PWR06") (unit 1)
@@
     (pin "2")
     (instances
-      (project "MySXSenors"
+      (project "MySXSensors"
         (path "/95f78fe7-75c4-427a-aee1-7170190425b2"
           (reference "C2") (unit 1)
@@
       (effects (font (size 1.27 1.27)))
     )
-    (property "Footprint" "MySXSenors:FE10-2" (at 97.79 125.73 0)
+    (property "Footprint" "MySXSensors:FE10-2" (at 97.79 125.73 0)
       (effects (font (size 1.27 1.27)) hide)
     )
@@
     (pin "10")
     (instances
-      (project "MySXSenors"
+      (project "MySXSensors"
         (path "/95f78fe7-75c4-427a-aee1-7170190425b2"
           (reference "X1") (unit 1)

Commit message: version 1.0
Connections:
- net D3_INT: now also J1.1 (Pin_1); no longer J1.5 (Pin_5)
- net GND: now also J1.4 (Pin_4), J2.3 (Pin_3); no longer J1.2 (Pin_2), J2.2 (Pin_2)
- net VRAW: now also J1.5 (Pin_5), J2.4 (Pin_4); no longer J1.1 (Pin_1), J2.1 (Pin_1)
- net at J1.3 (Pin_3): now also J2.2 (Pin_2); no longer J2.3 (Pin_3)
- new net: J1.2 (Pin_2), J2.1 (Pin_1)
Changed lines of the file:
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@@
+    (stroke (width 0) (type default))
+  )
+  (wire (pts (xy 161.925 126.365) (xy 160.02 126.365))
+    (stroke (width 0) (type default))
+  )
+  (wire (pts (xy 150.495 131.445) (xy 161.925 131.445))
+    (stroke (width 0) (type default))
+  )
+  (wire (pts (xy 160.02 110.49) (xy 161.925 110.49))
     (stroke (width 0) (type default))
   )
@@
     (stroke (width 0) (type default))
   )
+  (wire (pts (xy 195.58 53.975) (xy 195.58 43.18))
+    (stroke (width 0) (type default))
+  )
+  (wire (pts (xy 105.41 133.35) (xy 108.585 133.35))
+    (stroke (width 0.1524) (type solid))
+  )
+  (wire (pts (xy 124.46 71.12) (xy 124.46 48.26))
+    (stroke (width 0) (type default))
+  )
   (wire (pts (xy 151.765 133.985) (xy 161.925 133.985))
     (stroke (width 0) (type default))
   )
-  (wire (pts (xy 195.58 53.975) (xy 195.58 43.18))
-    (stroke (width 0) (type default))
-  )
-  (wire (pts (xy 105.41 133.35) (xy 108.585 133.35))
-    (stroke (width 0.1524) (type solid))
-  )
-  (wire (pts (xy 124.46 71.12) (xy 124.46 48.26))
-    (stroke (width 0) (type default))
-  )
   (wire (pts (xy 83.185 48.26) (xy 95.25 48.26))
     (stroke (width 0) (type default))
@@
     (stroke (width 0.1524) (type solid))
   )
+  (wire (pts (xy 161.925 128.905) (xy 160.02 128.905))
+    (stroke (width 0) (type default))
+  )
   (wire (pts (xy 95.25 78.74) (xy 97.79 78.74))
     (stroke (width 0) (type default))
@@
     (stroke (width 0) (type default))
   )
+  (wire (pts (xy 160.02 107.95) (xy 161.925 107.95))
+    (stroke (width 0) (type default))
+  )
   (wire (pts (xy 195.58 53.975) (xy 191.135 53.975))
     (stroke (width 0) (type default))
@@
     (stroke (width 0) (type default))
   )
+  (wire (pts (xy 83.185 59.055) (xy 83.185 55.88))
+    (stroke (width 0) (type default))
+  )
   (wire (pts (xy 105.41 118.11) (xy 108.585 118.11))
     (stroke (width 0.1524) (type solid))
@@
   (wire (pts (xy 105.41 115.57) (xy 108.585 115.57))
     (stroke (width 0.1524) (type solid))
-  )
-  (wire (pts (xy 150.495 131.445) (xy 161.925 131.445))
-    (stroke (width 0) (type default))
   )
   (wire (pts (xy 92.71 115.57) (xy 88.265 115.57))
@@
     )
   )
-  (global_label "VRAW" (shape input) (at 161.925 126.365 180) (fields_autoplaced)
-    (effects (font (size 1.27 1.27)) (justify right))
-    (property "Intersheetrefs" "${INTERSHEET_REFS}" (at 154.0412 126.365 0)
-      (effects (font (size 1.27 1.27)) (justify right) hide)
-    )
-  )
-  (global_label "VRAW" (shape input) (at 161.925 107.95 180) (fields_autoplaced)
-    (effects (font (size 1.27 1.27)) (justify right))
-    (property "Intersheetrefs" "${INTERSHEET_REFS}" (at 154.0412 107.95 0)
+  (global_label "VRAW" (shape input) (at 160.02 126.365 180) (fields_autoplaced)
+    (effects (font (size 1.27 1.27)) (justify right))
+    (property "Intersheetrefs" "${INTERSHEET_REFS}" (at 152.1362 126.365 0)
+      (effects (font (size 1.27 1.27)) (justify right) hide)
+    )
+  )
+  (global_label "VRAW" (shape input) (at 160.02 107.95 180) (fields_autoplaced)
+    (effects (font (size 1.27 1.27)) (justify right))
+    (property "Intersheetrefs" "${INTERSHEET_REFS}" (at 152.1362 107.95 0)
       (effects (font (size 1.27 1.27)) (justify right) hide)
     )
@@
     )
   )
-  (symbol (lib_id "power:GND") (at 161.925 128.905 270) (unit 1)
+  (symbol (lib_id "power:GND") (at 160.02 128.905 270) (unit 1)
     (in_bom yes) (on_board yes) (dnp no) (fields_autoplaced)
-    (property "Reference" "#PWR08" (at 155.575 128.905 0)
-      (effects (font (size 1.27 1.27)) hide)
-    )
-    (property "Value" "GND" (at 158.75 128.905 90)
+    (property "Reference" "#PWR08" (at 153.67 128.905 0)
+      (effects (font (size 1.27 1.27)) hide)
+    )
+    (property "Value" "GND" (at 156.845 128.905 90)
       (effects (font (size 1.27 1.27)) (justify right))
     )
-    (property "Footprint" "" (at 161.925 128.905 0)
-      (effects (font (size 1.27 1.27)) hide)
-    )
-    (property "Datasheet" "" (at 161.925 128.905 0)
+    (property "Footprint" "" (at 160.02 128.905 0)
+      (effects (font (size 1.27 1.27)) hide)
+    )
+    (property "Datasheet" "" (at 160.02 128.905 0)
       (effects (font (size 1.27 1.27)) hide)
     )
@@
     )
   )
-  (symbol (lib_id "Connector_Generic:Conn_01x04") (at 167.005 128.905 0) (unit 1)
-    (in_bom yes) (on_board yes) (dnp no) (fields_autoplaced)
-    (property "Reference" "J2" (at 170.18 128.905 0)
-      (effects (font (size 1.27 1.27)) (justify left))
-    )
-    (property "Value" "UART" (at 170.18 131.445 0)
-      (effects (font (size 1.27 1.27)) (justify left))
-    )
-    (property "Footprint" "Connector_PinHeader_2.54mm:PinHeader_1x04_P2.54mm_Horizontal" (at 167.005 128.905 0)
-      (effects (font (size 1.27 1.27)) hide)
-    )
-    (property "Datasheet" "~" (at 167.005 128.905 0)
+  (symbol (lib_id "Connector_Generic:Conn_01x04") (at 167.005 131.445 0) (mirror x) (unit 1)
+    (in_bom yes) (on_board yes) (dnp no)
+    (property "Reference" "J2" (at 170.18 131.445 0)
+      (effects (font (size 1.27 1.27)) (justify left))
+    )
+    (property "Value" "UART" (at 170.18 128.905 0)
+      (effects (font (size 1.27 1.27)) (justify left))
+    )
+    (property "Footprint" "Connector_PinHeader_2.54mm:PinHeader_1x04_P2.54mm_Horizontal" (at 167.005 131.445 0)
+      (effects (font (size 1.27 1.27)) hide)
+    )
+    (property "Datasheet" "~" (at 167.005 131.445 0)
       (effects (font (size 1.27 1.27)) hide)
     )
@@
     )
   )
-  (symbol (lib_id "power:GND") (at 161.925 110.49 270) (unit 1)
+  (symbol (lib_id "power:GND") (at 160.02 110.49 270) (unit 1)
     (in_bom yes) (on_board yes) (dnp no) (fields_autoplaced)
-    (property "Reference" "#PWR07" (at 155.575 110.49 0)
-      (effects (font (size 1.27 1.27)) hide)
-    )
-    (property "Value" "GND" (at 158.75 110.49 90)
+    (property "Reference" "#PWR07" (at 153.67 110.49 0)
+      (effects (font (size 1.27 1.27)) hide)
+    )
+    (property "Value" "GND" (at 156.845 110.49 90)
       (effects (font (size 1.27 1.27)) (justify right))
     )
-    (property "Footprint" "" (at 161.925 110.49 0)
-      (effects (font (size 1.27 1.27)) hide)
-    )
-    (property "Datasheet" "" (at 161.925 110.49 0)
+    (property "Footprint" "" (at 160.02 110.49 0)
+      (effects (font (size 1.27 1.27)) hide)
+    )
+    (property "Datasheet" "" (at 160.02 110.49 0)
       (effects (font (size 1.27 1.27)) hide)
     )
@@
     )
   )
-  (symbol (lib_id "power:GND") (at 83.185 55.88 0) (unit 1)
+  (symbol (lib_id "power:GND") (at 83.185 59.055 0) (unit 1)
     (in_bom yes) (on_board yes) (dnp no) (fields_autoplaced)
-    (property "Reference" "#PWR04" (at 83.185 62.23 0)
-      (effects (font (size 1.27 1.27)) hide)
-    )
-    (property "Value" "GND" (at 83.185 60.325 0)
+    (property "Reference" "#PWR04" (at 83.185 65.405 0)
+      (effects (font (size 1.27 1.27)) hide)
+    )
+    (property "Value" "GND" (at 83.185 63.5 0)
       (effects (font (size 1.27 1.27)))
     )
-    (property "Footprint" "" (at 83.185 55.88 0)
-      (effects (font (size 1.27 1.27)) hide)
-    )
-    (property "Datasheet" "" (at 83.185 55.88 0)
+    (property "Footprint" "" (at 83.185 59.055 0)
+      (effects (font (size 1.27 1.27)) hide)
+    )
+    (property "Datasheet" "" (at 83.185 59.055 0)
       (effects (font (size 1.27 1.27)) hide)
     )
@@
     )
   )
-  (symbol (lib_id "Connector_Generic:Conn_01x05") (at 167.005 113.03 0) (unit 1)
-    (in_bom yes) (on_board yes) (dnp no) (fields_autoplaced)
-    (property "Reference" "J1" (at 169.545 111.76 0)
-      (effects (font (size 1.27 1.27)) (justify left))
-    )
-    (property "Value" "LD2410B" (at 169.545 114.3 0)
-      (effects (font (size 1.27 1.27)) (justify left))
-    )
+  (symbol (lib_id "Connector_Generic:Conn_01x05") (at 167.005 113.03 0) (mirror x) (unit 1)
+    (in_bom yes) (on_board yes) (dnp no)
+    (property "Reference" "J1" (at 169.545 114.3 0)
+      (effects (font (size 1.27 1.27)) (justify left))
+    )
+    (property "Value" "LD2410B" (at 169.545 111.76 0)
+      (effects (font (size 1.27 1.27)) (justify left))
+    )
